File: beerodul.kicad_pcb (KiCad board)
At the start: 2 copper layers, 97.5 x 50.9 mm, 0 parts

Commit message: Sexy rexy
Parts:
- added BT1: Battery_Cell, Battery:BatteryHolder_Keystone_103_1x20mm, B.Cu at (148.0, 79.0)
- added G***: LOGO, graphics:bsides, F.Cu at (156.2, 78.2)
Routing:
- added copper zone on F.Cu, net Net-(BT1-Pad1)
Other:
- outline, holes or cut-outs redrawn

Commit message: Work work
Parts:
- added BZ1: Buzzer, Buzzer_Beeper:Buzzer_12x9.5RM7.6, B.Cu at (171.5, 78.7)
- added REF**: MountingHole_3.2mm_M3, MountingHole:MountingHole_3.2mm_M3, F.Cu at (182.9, 78.7)
- moved BT1 14.7 mm to (133.3, 78.7)
- moved G*** 5.70 mm to (162.0, 78.1)
Routing:
- net Net-(BZ1-Pad1): track 0.00 -> 35.6 mm, vias 0 -> 8
- net Net-(BT1-Pad2): track 0.00 -> 11.3 mm
- added copper zone on B.Cu, net Net-(BZ1-Pad1)
Changed lines of the file:
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@@
   (general
     (thickness 1.6)
-    (drawings 12)
-    (tracks 0)
+    (drawings 13)
+    (tracks 17)
     (zones 0)
-    (modules 2)
-    (nets 3)
+    (modules 4)
+    (nets 4)
   )
   (page A4)
   (layers
     (0 F.Cu signal hide)
-    (31 B.Cu signal)
+    (31 B.Cu signal hide)
     (32 B.Adhes user)
     (33 F.Adhes user)
@@
     (37 F.SilkS user)
     (38 B.Mask user)
-    (39 F.Mask user)
+    (39 F.Mask user hide)
     (40 Dwgs.User user)
     (41 Cmts.User user)
@@
   (net 1 "Net-(BT1-Pad2)")
   (net 2 "Net-(BT1-Pad1)")
+  (net 3 "Net-(BZ1-Pad1)")
   (net_class Default "This is the default net class."
     (clearance 0.2)
@@
     (add_net "Net-(BT1-Pad1)")
     (add_net "Net-(BT1-Pad2)")
+    (add_net "Net-(BZ1-Pad1)")
   )
   (module Battery:BatteryHolder_Keystone_103_1x20mm (layer B.Cu)
-    (at 148 79)
+    (at 133.35 78.74)
     (descr http://www.keyelco.com/product-pdf.cfm?p=719)
     (tags "Keystone type 103 battery holder")
@@
   )
   (module graphics:bsides (layer F.Cu)
-    (at 156.25 78.25)
+    (at 161.9504 78.0796)
     (fp_text reference G*** (at 0 0) (layer F.SilkS) hide
       (effects (font (size 1.524 1.524) (thickness 0.3)))
@@
       (xy -7.373733 -12.4427) (xy -7.051259 -12.560007) (xy -6.732191 -12.575157) (xy -6.396955 -12.489236)) (layer F.SilkS) (width 0.01))
   )
+  (module Buzzer_Beeper:Buzzer_12x9.5RM7.6 (layer B.Cu)
+    (at 171.47 78.74 180)
+    (descr "Generic Buzzer, D12mm height 9.5mm with RM7.6mm")
+    (tags buzzer)
+    (fp_text reference BZ1 (at 3.8 7.2 180) (layer B.SilkS)
+      (effects (font (size 1 1) (thickness 0.15)) (justify mirror))
+    )
+    (fp_text value Buzzer (at 3.8 -7.4 180) (layer B.Fab)
+      (effects (font (size 1 1) (thickness 0.15)) (justify mirror))
+    )
+    (fp_text user + (at -0.01 2.54 180) (layer B.Fab)
+      (effects (font (size 1 1) (thickness 0.15)) (justify mirror))
+    )
+    (fp_text user + (at -0.01 2.54 180) (layer B.SilkS)
+      (effects (font (size 1 1) (thickness 0.15)) (justify mirror))
+    )
+    (fp_text user %R (at 3.8 4 180) (layer B.Fab)
+      (effects (font (size 1 1) (thickness 0.15)) (justify mirror))
+    )
+    (fp_circle (center 3.8 0) (end 10.05 0) (layer B.CrtYd) (width 0.05))
+    (fp_circle (center 3.8 0) (end 9.8 0) (layer B.Fab) (width 0.1))
+    (fp_circle (center 3.8 0) (end 4.8 0) (layer B.Fab) (width 0.1))
+    (fp_circle (center 3.8 0) (end 9.9 0) (layer B.SilkS) (width 0.12))
+    (pad 1 thru_hole rect (at 0 0 180) (size 2 2) (drill 1) (layers *.Cu *.Mask)
+      (net 3 "Net-(BZ1-Pad1)"))
+    (pad 2 thru_hole circle (at 7.6 0 180) (size 2 2) (drill 1) (layers *.Cu *.Mask)
+      (net 1 "Net-(BT1-Pad2)"))
+    (model ${KISYS3DMOD}/Buzzer_Beeper.3dshapes/Buzzer_12x9.5RM7.6.wrl
+      (at (xyz 0 0 0))
+      (scale (xyz 1 1 1))
+      (rotate (xyz 0 0 0))
+    )
+  )
+  (module MountingHole:MountingHole_3.2mm_M3 (layer F.Cu)
+    (at 182.88 78.74)
+    (descr "Mounting Hole 3.2mm, no annular, M3")
+    (tags "mounting hole 3.2mm no annular m3")
+    (attr virtual)
+    (fp_text reference REF** (at 0 -4.2) (layer F.SilkS)
+      (effects (font (size 1 1) (thickness 0.15)))
+    )
+    (fp_text value MountingHole_3.2mm_M3 (at 0 4.2) (layer F.Fab)
+      (effects (font (size 1 1) (thickness 0.15)))
+    )
+    (fp_circle (center 0 0) (end 3.45 0) (layer F.CrtYd) (width 0.05))
+    (fp_circle (center 0 0) (end 3.2 0) (layer Cmts.User) (width 0.15))
+    (fp_text user %R (at 0.3 0) (layer F.Fab)
+      (effects (font (size 1 1) (thickness 0.15)))
+    )
+    (pad 1 np_thru_hole circle (at 0 0) (size 3.2 3.2) (drill 3.2) (layers *.Cu *.Mask))
+  )
+  (gr_poly (pts (xy 125.73 68.58) (xy 125.73 88.9) (xy 130.175 88.9) (xy 130.175 68.58)) (layer F.Mask) (width 0.15))
   (gr_arc (start 140 102) (end 135 97) (angle 53.1) (layer Edge.Cuts) (width 0.2))
   (gr_arc (start 140 56) (end 135 61) (angle -53.1) (layer Edge.Cuts) (width 0.2))
@@
   (gr_arc (start 183 69) (end 189 69) (angle -90) (layer Edge.Cuts) (width 0.2))
   (gr_arc (start 124.5 69) (end 125.5 69) (angle -53.13010235) (layer Edge.Cuts) (width 0.2))
+  (segment (start 171.47 78.74) (end 160.19 78.74) (width 0.25) (layer B.Cu) (net 1))
+  (via (at 130.81 69.85) (size 0.8) (drill 0.4) (layers F.Cu B.Cu) (net 3))
+  (via (at 130.81 72.39) (size 0.8) (drill 0.4) (layers F.Cu B.Cu) (net 3))
+  (via (at 130.81 74.93) (size 0.8) (drill 0.4) (layers F.Cu B.Cu) (net 3))
+  (via (at 130.81 77.47) (size 0.8) (drill 0.4) (layers F.Cu B.Cu) (net 3))
+  (via (at 130.81 80.01) (size 0.8) (drill 0.4) (layers F.Cu B.Cu) (net 3))
+  (via (at 130.81 82.55) (size 0.8) (drill 0.4) (layers F.Cu B.Cu) (net 3))
+  (via (at 130.81 85.09) (size 0.8) (drill 0.4) (layers F.Cu B.Cu) (net 3))
+  (via (at 130.81 87.63) (size 0.8) (drill 0.4) (layers F.Cu B.Cu) (net 3))
+  (segment (start 130.81 69.85) (end 126.365 69.85) (width 0.5) (layer F.Cu) (net 3))
+  (segment (start 130.81 72.39) (end 126.365 72.39) (width 0.5) (layer F.Cu) (net 3))
+  (segment (start 130.81 74.93) (end 126.365 74.93) (width 0.5) (layer F.Cu) (net 3))
+  (segment (start 130.81 77.47) (end 126.365 77.47) (width 0.5) (layer F.Cu) (net 3))
+  (segment (start 130.81 80.01) (end 126.365 80.01) (width 0.5) (layer F.Cu) (net 3))
+  (segment (start 130.81 82.55) (end 126.365 82.55) (width 0.5) (layer F.Cu) (net 3))
+  (segment (start 130.81 85.09) (end 126.365 85.09) (width 0.5) (layer F.Cu) (net 3))
+  (segment (start 130.81 87.63) (end 126.365 87.63) (width 0.5) (layer F.Cu) (net 3))
   (zone (net 2) (net_name "Net-(BT1-Pad1)") (layer F.Cu) (hatch edge 0.508)
     (connect_pads (clearance 0.508))
@@
       )
     )
+  )
+  (zone (net 3) (net_name "Net-(BZ1-Pad1)") (layer B.Cu) (hatch edge 0.508)
+    (connect_pads (clearance 0.508))
+    (min_thickness 0.254)
+    (fill yes (arc_segments 16) (thermal_gap 0.508) (thermal_bridge_width 0.508))
+    (polygon
+      (pts
+        (xy 88.9 50.8) (xy 88.9 107.95) (xy 190.5 107.315) (xy 190.5 50.165)
+      )
+    )

Commit message: 3 days
Parts:
- removed the G*** at (162.0, 78.1)
- removed the REF** at (182.9, 78.7)
- added G***: LOGO, graphics:bsides2, F.Cu at (159.9, 78.1)
- added REF**: MountingHole_5mm, MountingHole:MountingHole_5mm, F.Cu at (184.2, 78.7)
Routing:
- net Net-(BT1-Pad2): track 11.3 -> 10.0 mm
Other:
- board text added: "BSidesLjubljana::0x7E3"
- board text added: "CUT OUT"

Commit message: Mid day edit
Routing:
- net Net-(BZ1-Pad1): track 35.6 -> 65.9 mm
Changed lines of the file:
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@@
-(kicad_pcb (version 20171130) (host pcbnew "(5.0.2)-1")
+(kicad_pcb (version 20171130) (host pcbnew 5.0.2)
   (general
     (thickness 1.6)
-    (drawings 15)
-    (tracks 17)
+    (drawings 16)
+    (tracks 20)
     (zones 0)
     (modules 4)
@@
     (pad 1 np_thru_hole circle (at 0 0) (size 5 5) (drill 5) (layers *.Cu *.Mask))
   )
+  (gr_line (start 139.5 87) (end 179.5 87) (layer F.SilkS) (width 0.7))
   (gr_text "CUT OUT" (at 114.3 78.74) (layer F.Fab)
     (effects (font (size 1.5 1.5) (thickness 0.3)))
   )
-  (gr_text BSidesLjubljana::0x7E3 (at 167.64 90.17) (layer F.SilkS)
+  (gr_text BSidesLjubljana::0x7E3 (at 163 90.17) (layer F.SilkS)
     (effects (font (size 2 2) (thickness 0.3)))
   )
@@
   (segment (start 130.81 85.09) (end 126.365 85.09) (width 0.5) (layer F.Cu) (net 3))
   (segment (start 130.81 87.63) (end 126.365 87.63) (width 0.5) (layer F.Cu) (net 3))
+  (segment (start 130.81 87.63) (end 130.81 92.19) (width 0.25) (layer F.Cu) (net 3))
+  (segment (start 130.81 92.19) (end 126 97) (width 0.25) (layer F.Cu) (net 3))
+  (segment (start 126 97) (end 107 97) (width 0.25) (layer F.Cu) (net 3))
   (zone (net 2) (net_name "Net-(BT1-Pad1)") (layer F.Cu) (hatch edge 0.508)
     (connect_pads (clearance 0.508))

Commit message: Add renders
Routing:
- net Net-(BZ1-Pad1): track 65.9 -> 103.4 mm
Other:
- board text added: "16th March 2019 Ljubljana, Slovenia"
Changed lines of the file:
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@@
-(kicad_pcb (version 20171130) (host pcbnew 5.0.2)
+(kicad_pcb (version 20171130) (host pcbnew "(5.0.2)-1")
   (general
     (thickness 1.6)
-    (drawings 16)
-    (tracks 20)
+    (drawings 19)
+    (tracks 40)
     (zones 0)
     (modules 4)
@@
   (page A4)
   (layers
-    (0 F.Cu signal hide)
+    (0 F.Cu signal)
     (31 B.Cu signal hide)
     (32 B.Adhes user)
@@
     (37 F.SilkS user)
     (38 B.Mask user)
-    (39 F.Mask user hide)
+    (39 F.Mask user)
     (40 Dwgs.User user)
     (41 Cmts.User user)
@@
     (visible_elements 7FFFFFFF)
     (pcbplotparams
-      (layerselection 0x010fc_ffffffff)
-      (usegerberextensions false)
+      (layerselection 0x012f0_ffffffff)
+      (usegerberextensions true)
       (usegerberattributes false)
       (usegerberadvancedattributes false)
@@
       (outputformat 1)
       (mirror false)
-      (drillshape 1)
+      (drillshape 0)
       (scaleselection 1)
-      (outputdirectory ""))
+      (outputdirectory "gerber/"))
   )
   (net 0 "")
@@
     (pad 1 np_thru_hole circle (at 0 0) (size 5 5) (drill 5) (layers *.Cu *.Mask))
   )
-  (gr_line (start 139.5 87) (end 179.5 87) (layer F.SilkS) (width 0.7))
-  (gr_text "CUT OUT" (at 114.3 78.74) (layer F.Fab)
+  (gr_text "16th March 2019\nLjubljana, Slovenia" (at 102.87 66.04 -135) (layer F.Cu)
+    (effects (font (size 1 1) (thickness 0.25)))
+  )
+  (gr_line (start 139.6492 86.487) (end 139.3698 87.6808) (layer F.SilkS) (width 0.65))
+  (gr_line (start 179.578 86.5886) (end 179.58816 87.63) (layer F.SilkS) (width 0.7))
+  (gr_line (start 139.4714 87.6554) (end 179.58308 87.6554) (layer F.SilkS) (width 0.7))
+  (gr_text "CUT OUT" (at 114.3 78.74) (layer Cmts.User)
     (effects (font (size 1.5 1.5) (thickness 0.3)))
   )
-  (gr_text BSidesLjubljana::0x7E3 (at 163 90.17) (layer F.SilkS)
+  (gr_text BSidesLjubljana::0x7E3 (at 162.56 90.932) (layer F.SilkS)
     (effects (font (size 2 2) (thickness 0.3)))
   )
@@
   (segment (start 130.81 87.63) (end 130.81 92.19) (width 0.25) (layer F.Cu) (net 3))
   (segment (start 130.81 92.19) (end 126 97) (width 0.25) (layer F.Cu) (net 3))
-  (segment (start 126 97) (end 107 97) (width 0.25) (layer F.Cu) (net 3))
+  (segment (start 121.92 97) (end 119.86 97) (width 0.25) (layer F.Cu) (net 3))
+  (segment (start 119.86 97) (end 118.9 97) (width 0.25) (layer F.Cu) (net 3))
+  (segment (start 118.9 97) (end 115.57 100.33) (width 0.25) (layer F.Cu) (net 3))
+  (segment (start 124.46 97) (end 123.67 97) (width 0.25) (layer F.Cu) (net 3))
+  (segment (start 124.46 97) (end 121.92 97) (width 0.25) (layer F.Cu) (net 3))
+  (segment (start 126 97) (end 124.46 97) (width 0.25) (layer F.Cu) (net 3))
+  (segment (start 123.67 97) (end 120.65 93.98) (width 0.25) (layer F.Cu) (net 3))
+  (segment (start 123.67 97) (end 122.71 97) (width 0.25) (layer F.Cu) (net 3))
+  (segment (start 122.71 97) (end 119.38 100.33) (width 0.25) (layer F.Cu) (net 3))
+  (segment (start 115.57 97) (end 114.78 97) (width 0.25) (layer F.Cu) (net 3))
+  (segment (start 114.78 97) (end 111.76 93.98) (width 0.25) (layer F.Cu) (net 3))
+  (segment (start 114.78 97) (end 113.82 97) (width 0.25) (layer F.Cu) (net 3))
+  (segment (start 113.82 97) (end 110.49 100.33) (width 0.25) (layer F.Cu) (net 3))
+  (segment (start 111.76 97) (end 110.97 97) (width 0.25) (layer F.Cu) (net 3))
+  (segment (start 111.76 97) (end 107 97) (width 0.25) (layer F.Cu) (net 3))
+  (segment (start 115.57 97) (end 111.76 97) (width 0.25) (layer F.Cu) (net 3))
+  (segment (start 110.97 97) (end 109.22 95.25) (width 0.25) (layer F.Cu) (net 3))
+  (segment (start 118.11 97) (end 117.32 97) (width 0.25) (layer F.Cu) (net 3))
+  (segment (start 118.11 97) (end 115.57 97) (width 0.25) (layer F.Cu) (net 3))
+  (segment (start 121.92 97) (end 118.11 97) (width 0.25) (layer F.Cu) (net 3))
+  (segment (start 117.32 97) (end 114.3 93.98) (width 0.25) (layer F.Cu) (net 3))
   (zone (net 2) (net_name "Net-(BT1-Pad1)") (layer F.Cu) (hatch edge 0.508)
     (connect_pads (clearance 0.508))
@@
       )
     )
+  )
+  (zone (net 0) (net_name "") (layer B.Cu) (hatch edge 0.508)
+    (connect_pads (clearance 0.508))
+    (min_thickness 0.254)
+    (keepout (tracks not_allowed) (vias not_allowed) (copperpour not_allowed))
+    (fill (arc_segments 16) (thermal_gap 0.508) (thermal_bridge_width 0.508))
+    (polygon
+      (pts
+        (xy 177.8 60.96) (xy 177.8 99.06) (xy 190.5 99.06) (xy 190.5 60.96)
+      )
+    )
